File: LEDBoard/LED-Nicola/Led_Board.sch (KiCad schematic (older format))
At the start: 36 parts, among them J1 MOUNTING_HOLE, J10 CONN_01X02, J11 LED CONN 01X16, J12 CONN_01X02, J13 LED CONN 01X04, J2 MOUNTING_HOLE, J3 MOUNTING_HOLE, J4 MOUNTING_HOLE, J5 Arduino CONN 01X04, J6 Arduino CONN_01X04, J7 Arduino CONN_01X06, J8 VD 0 CONN_01X02, J9 CONN_01X02, Q1 MMBT2222ALT1G, U1 SSR

Commit message: Made a couple final changes to the LED Board- Should be good to go
Parts:
- added J101: CONN_01X01, hyperCustom:CONN_PHOENIX_1844210_1PIN, symbol CONN_01X01
Connections:
- net GND: now also J101.1 (P1)
Changed lines of the file:
@@
 Text Label 3900 6650 3    60   ~ 0
 ArduinoLED
+$Comp
+L CONN_01X01 J101
+U 1 1 597FCC23
+P 2400 3600
+F 0 "J101" H 2400 3700 50  0000 C CNN
+F 1 "CONN_01X01" V 2500 3600 50  0000 C CNN
+F 2 "hyperCustom:CONN_PHOENIX_1844210_1PIN" H 2400 3600 50  0001 C CNN
+F 3 "" H 2400 3600 50  0001 C CNN
+	1    2400 3600
+	-1   0    0    1
+$EndComp
+$Comp
+L GND #PWR101
+U 1 1 597FD493
+P 2600 3600
+F 0 "#PWR101" H 2600 3350 50  0001 C CNN
+F 1 "GND" H 2600 3450 50  0000 C CNN
+F 2 "" H 2600 3600 50  0001 C CNN
+F 3 "" H 2600 3600 50  0001 C CNN
+	1    2600 3600
+	1    0    0    -1
+$EndComp
 $EndSCHEMATC

Commit message: Added Connector
Parts:
- removed J101: CONN_01X01, hyperCustom:CONN_PHOENIX_1844210_1PIN, symbol CONN_01X01
- removed J5: Arduino CONN 01X04, hyperCustom:CONN_PHOENIX_1844236_4PIN, symbol CONN_01X04
- added J5: CONN_01X06, hyperCustom:CONN_PHOENIX_1844252_6PIN, symbol CONN_01X06
Connections:
- net 24V: now also J5.2 (P2)
- net 5V0: now also J5.3 (P3)
- net A0: now also J5.1 (P1)
- net GND: now also J5.5 (P5)
- net Transistor: now also J5.4 (P4)
Changed lines of the file:
@@
 LIBS:contrib
 LIBS:valves
+LIBS:KiCAD_Tutorial
+LIBS:5vregulatortab
+LIBS:ssr
+LIBS:SSRBoard-cache
+LIBS:SSRBoard-rescue
+LIBS:Arduino_Uno_R3_From_Scratch
+LIBS:Arduino_Uno_R3_From_Scratch-cache
+LIBS:MFN_Atmel
+LIBS:xtr117
+LIBS:mmbt2222alt1g
+LIBS:VO14642AABTR
 LIBS:Led_Board-cache
 EELAYER 25 0
@@
 Text Label 5350 5050 3    60   ~ 0
 VDI2
-$Comp
-L CONN_01X04 J5
-U 1 1 5979ADB2
-P 2400 2200
-F 0 "J5" H 2500 2150 50  0000 C CNN
-F 1 "Arduino CONN 01X04" H 2850 2050 50  0000 C CNN
-F 2 "hyperCustom:CONN_PHOENIX_1844236_4PIN" H 2400 2200 50  0001 C CNN
-F 3 "" H 2400 2200 50  0001 C CNN
-F 4 "277-2419-ND" H 2400 2200 60  0001 C CNN "Digikey PN"
-F 5 "Phoenix" H 2400 2200 60  0001 C CNN "Mfg. "
-F 6 "1844236" H 2400 2200 60  0001 C CNN "Mfg. PN"
-	1    2400 2200
-	-1   0    0    1
-$EndComp
 $Comp
 L CONN_01X04 J6
@@
 ArduinoLED
 $Comp
-L CONN_01X01 J101
-U 1 1 597FCC23
-P 2400 3600
-F 0 "J101" H 2400 3700 50  0000 C CNN
-F 1 "CONN_01X01" V 2500 3600 50  0000 C CNN
-F 2 "hyperCustom:CONN_PHOENIX_1844210_1PIN" H 2400 3600 50  0001 C CNN
-F 3 "" H 2400 3600 50  0001 C CNN
-	1    2400 3600
+L GND #PWR01
+U 1 1 597FD493
+P 2600 1950
+F 0 "#PWR01" H 2600 1700 50  0001 C CNN
+F 1 "GND" H 2600 1800 50  0000 C CNN
+F 2 "" H 2600 1950 50  0001 C CNN
+F 3 "" H 2600 1950 50  0001 C CNN
+	1    2600 1950
 	-1   0    0    1
 $EndComp
 $Comp
-L GND #PWR101
-U 1 1 597FD493
-P 2600 3600
-F 0 "#PWR101" H 2600 3350 50  0001 C CNN
-F 1 "GND" H 2600 3450 50  0000 C CNN
-F 2 "" H 2600 3600 50  0001 C CNN
-F 3 "" H 2600 3600 50  0001 C CNN
-	1    2600 3600
-	1    0    0    -1
+L CONN_01X06 J5
+U 1 1 598146EF
+P 2400 2100
+F 0 "J5" H 2400 2450 50  0000 C CNN
+F 1 "CONN_01X06" V 2500 2100 50  0000 C CNN
+F 2 "hyperCustom:CONN_PHOENIX_1844252_6PIN" H 2400 2100 50  0001 C CNN
+F 3 "" H 2400 2100 50  0001 C CNN
+	1    2400 2100
+	-1   0    0    1
 $EndComp
 $EndSCHEMATC

Commit message: Final Changes
Good to go. Added the correct 5 pin connector.
Parts:
- removed J5: CONN_01X06, hyperCustom:CONN_PHOENIX_1844252_6PIN, symbol CONN_01X06
- added J101: CONN_01X05, hyperCustom:CONN_PHOENIX_1844252_5PIN, symbol CONN_01X05
Connections:
- net 24V: now also J101.2 (P2)
- net 5V0: now also J101.3 (P3)
- net A0: now also J101.1 (P1)
- net GND: now also J101.5 (P5)
- net Transistor: now also J101.4 (P4)
Other:
- moved on the sheet: J7
Changed lines of the file:
@@
 LIBS:contrib
 LIBS:valves
-LIBS:KiCAD_Tutorial
-LIBS:5vregulatortab
-LIBS:ssr
-LIBS:SSRBoard-cache
-LIBS:SSRBoard-rescue
-LIBS:Arduino_Uno_R3_From_Scratch
-LIBS:Arduino_Uno_R3_From_Scratch-cache
-LIBS:MFN_Atmel
-LIBS:xtr117
-LIBS:mmbt2222alt1g
-LIBS:VO14642AABTR
 LIBS:Led_Board-cache
 EELAYER 25 0
@@
 	8850 4800 8850 4900
 Wire Wire Line
-	2600 2350 2850 2350
-Wire Wire Line
 	2600 2450 2850 2450
 Wire Wire Line
@@
 	2600 2750 2850 2750
 Wire Wire Line
-	2600 2850 2850 2850
-Wire Wire Line
-	2600 2950 2850 2950
-Text Label 2850 2350 0    60   ~ 0
+	2600 3050 2850 3050
+Wire Wire Line
+	2600 3150 2850 3150
+Text Label 2900 2000 0    60   ~ 0
 A0
 Text Label 2850 2450 0    60   ~ 0
@@
 Text Label 2850 2750 0    60   ~ 0
 A4
-Text Label 2850 2850 0    60   ~ 0
+Text Label 2850 3050 0    60   ~ 0
 A5
-Text Label 2850 2950 0    60   ~ 0
+Text Label 2850 3150 0    60   ~ 0
 A6
-Text Label 2600 2050 0    60   ~ 0
+Text Label 2650 1700 0    60   ~ 0
 Transistor
 Wire Wire Line
-	2600 3050 2850 3050
+	2600 3250 2850 3250
 Text Label 2850 2550 0    60   ~ 0
 A2
-Text Label 2600 2250 0    60   ~ 0
+Text Label 2650 1900 0    60   ~ 0
 24V
 $Comp
@@
 $EndComp
 Wire Wire Line
-	2600 3150 2850 3150
+	2600 3350 2850 3350
 $Comp
 L MOUNTING_HOLE J1
@@
 GND
 Wire Wire Line
-	2600 3250 2850 3250
+	2600 3450 2850 3450
 Wire Wire Line
 	7650 4500 7650 4250
@@
 	5800 1000 5800 1150
 Wire Wire Line
-	2600 3350 2850 3350
-Text Label 2600 2150 0    60   ~ 0
+	2600 3550 2850 3550
+Text Label 2650 1800 0    60   ~ 0
 5V0
-Text Label 2850 3050 0    60   ~ 0
+Text Label 2850 3250 0    60   ~ 0
 A7
-Text Label 2850 3150 0    60   ~ 0
+Text Label 2850 3350 0    60   ~ 0
 A8
 $Comp
 L CONN_01X06 J7
 U 1 1 597E4F88
-P 2400 3100
-F 0 "J7" H 2500 2950 50  0000 C CNN
-F 1 "Arduino CONN_01X06" H 2850 2850 50  0000 C CNN
-F 2 "hyperCustom:CONN_PHOENIX_1844252_6PIN" H 2400 3100 50  0001 C CNN
-F 3 "" H 2400 3100 50  0001 C CNN
-F 4 "277-2427-ND" H 2400 3100 60  0001 C CNN "Digikey PN"
-F 5 "Phoenix" H 2400 3100 60  0001 C CNN "Mfg. "
-F 6 "1844525" H 2400 3100 60  0001 C CNN "Mfg. PN"
-	1    2400 3100
+P 2400 3300
+F 0 "J7" H 2500 3150 50  0000 C CNN
+F 1 "Arduino CONN_01X06" H 2850 3050 50  0000 C CNN
+F 2 "hyperCustom:CONN_PHOENIX_1844252_6PIN" H 2400 3300 50  0001 C CNN
+F 3 "" H 2400 3300 50  0001 C CNN
+F 4 "277-2427-ND" H 2400 3300 60  0001 C CNN "Digikey PN"
+F 5 "Phoenix" H 2400 3300 60  0001 C CNN "Mfg. "
+F 6 "1844525" H 2400 3300 60  0001 C CNN "Mfg. PN"
+	1    2400 3300
 	-1   0    0    1
 $EndComp
@@
 Text Label 1500 5300 2    60   ~ 0
 GND
-Text Label 2850 3250 0    60   ~ 0
+Text Label 2850 3450 0    60   ~ 0
 5V
-Text Label 2850 3350 0    60   ~ 0
+Text Label 2850 3550 0    60   ~ 0
 ArduinoLED
 $Comp
@@
 ArduinoLED
 $Comp
-L GND #PWR01
+L GND #PWR101
 U 1 1 597FD493
-P 2600 1950
-F 0 "#PWR01" H 2600 1700 50  0001 C CNN
-F 1 "GND" H 2600 1800 50  0000 C CNN
-F 2 "" H 2600 1950 50  0001 C CNN
-F 3 "" H 2600 1950 50  0001 C CNN
-	1    2600 1950
+P 2650 1600
+F 0 "#PWR101" H 2650 1350 50  0001 C CNN
+F 1 "GND" H 2650 1450 50  0000 C CNN
+F 2 "" H 2650 1600 50  0001 C CNN
+F 3 "" H 2650 1600 50  0001 C CNN
+	1    2650 1600
 	-1   0    0    1
 $EndComp
 $Comp
-L CONN_01X06 J5
-U 1 1 598146EF
-P 2400 2100
-F 0 "J5" H 2400 2450 50  0000 C CNN
-F 1 "CONN_01X06" V 2500 2100 50  0000 C CNN
-F 2 "hyperCustom:CONN_PHOENIX_1844252_6PIN" H 2400 2100 50  0001 C CNN
-F 3 "" H 2400 2100 50  0001 C CNN
-	1    2400 2100
+L CONN_01X05 J101
+U 1 1 598148B2
+P 2450 1800
+F 0 "J101" H 2450 2100 50  0000 C CNN
+F 1 "CONN_01X05" V 2550 1800 50  0000 C CNN
+F 2 "hyperCustom:CONN_PHOENIX_1844252_5PIN" H 2450 1800 50  0001 C CNN
+F 3 "" H 2450 1800 50  0001 C CNN
+F 4 "277-1610-ND" H 2450 1800 60  0001 C CNN "Digikey PN"
+	1    2450 1800
 	-1   0    0    1
 $EndComp
+Wire Wire Line
+	2650 2000 2900 2000
 $EndSCHEMATC
